Commit message: added files

File: p3dx_description/urdf/pioneer3dx.xacro (robot description, xacro)
@@ -92,5 +92,5 @@
 			<origin xyz="0 0 0" rpy="0 0 0" />
 			<geometry>
-				<box size="0 0 0" />
+				<box size="0.001 0.001 0.001" />
 			</geometry>
 		</collision>
@@ -125,5 +125,5 @@
 			<origin xyz="0 0 0" rpy="0 0 0" />
 			<geometry>
-				<box size="0 0 0" />
+				<box size="0.001 0.001 0.001" />
 			</geometry>
 		</collision>
@@ -188,5 +188,5 @@
 			<origin rpy="0 0 0" xyz="0 0 0" />
 			<geometry>
-				<box size="0 0 0" />
+				<box size="0.001 0.001 0.001" />
 			</geometry>
 		</collision>

File: p3dx_description/urdf/pioneer3dx_wheel.xacro (robot description, xacro)
@@ -18,5 +18,5 @@
 <robot xmlns:xacro="http://ros.org/wiki/xacro">
 	<!-- properties (constants) -->
-	<property name="M_PI" value="3.14159" />
+	<xacro:property name="M_PI" value="3.14159" />
 	<!-- right/left hubcap + wheel -->
 	<xacro:macro name="p3dx_wheel" params="suffix parent reflect">
@@ -71,5 +71,5 @@
 				<origin xyz="0 0 0" rpy="0 0 0" />
 				<geometry>
-					<box size="0 0 0" />
+					<box size="0.001 0.001 0.001" />
 				</geometry>
 			</collision>
